File: split/split.sch (KiCad schematic (older format))
At the start: 106 parts, among them K1 KEYSW, K10 KEYSW, K11 KEYSW, K12 KEYSW, K13 KEYSW, K14 KEYSW, K15 KEYSW, K16 KEYSW, K17 KEYSW, K18 KEYSW, K19 KEYSW, K2 KEYSW, K20 KEYSW, K21 KEYSW, K22 KEYSW, K23 KEYSW, K24 KEYSW, K25 KEYSW, K26 KEYSW, K27 KEYSW, K28 KEYSW, K29 KEYSW, K3 KEYSW, K30 KEYSW, K31 KEYSW, K32 KEYSW, K33 KEYSW, K34 KEYSW, K35 KEYSW, K36 KEYSW, K37 KEYSW, K38 KEYSW, K39 KEYSW, K4 KEYSW, K40 KEYSW, K41 KEYSW, K42 KEYSW, K43 KEYSW, K44 KEYSW, K45 KEYSW, K5 KEYSW, K6 KEYSW, K7 KEYSW, K8 KEYSW, K9 KEYSW, SW1 SW_PUSH, U1 ATMEGA32U4, X1 XTAL_GND

Commit message: init pcb layout
Parts:
- C1, C2, C3, C4, C5, C6, C7, C8: footprint (none) -> Capacitors:0805
- D1, D10, D11, D12, D13, D14, D15, D16, D17, D18, D19, D2, D20, D21, D22, D23, D24, D25, D26, D27, D28, D29, D3, D30, D31, D33, D34, D35, D36, D37, D38, D39, D4, D40, D41, D42, D43, D44, D45, D5, D6, D7, D8, D9: footprint (none) -> keyboard_parts:D_SOD123_axial
- D32: renamed from D?; footprint (none) -> keyboard_parts:D_SOD123_axial
- J1: renamed from J?; footprint (none) -> keyboard_parts:USB_miniB_hirose_5S8
- K1, K10, K11, K13, K14, K15, K16, K17, K18, K20, K21, K22, K23, K24, K25, K27, K28, K29, K30, K31, K32, K34, K35, K36, K37, K38, K39, K40, K41, K44, K45, K5, K6, K7, K9: footprint (none) -> MX_Alps_Hybrid:MX-1U-NoLED
- K12, K2, K4: footprint (none) -> MX_Alps_Hybrid:MX-1.25U-NoLED
- K19: footprint (none) -> MX_Alps_Hybrid:MX-2.25U-NoLED
- K26: footprint (none) -> MX_Alps_Hybrid:MX-2U-NoLED
- K3, K42: footprint (none) -> MX_Alps_Hybrid:MX-1.75U-NoLED
- K33, K43, K8: footprint (none) -> MX_Alps_Hybrid:MX-1.5U-NoLED
- R1, R2, R3: footprint 0603 -> Resistors:0805
- R4: renamed from R3; footprint 0603 -> Resistors:0805
- SW1: footprint (none) -> Button_Switch_SMD:SW_SPST_TL3342
- U1: footprint (none) -> Package_QFP:TQFP-44_10x10mm_P0.8mm
- X1: footprint (none) -> Crystal:Crystal_SMD_3225-4Pin_3.2x2.5mm
