File: split/split.kicad_pcb (KiCad board)
At the start: 2 copper layers, 106 parts, among them J1 USB_mini_micro_B, K1 KEYSW, K10 KEYSW, K11 KEYSW, K12 KEYSW, K13 KEYSW, K14 KEYSW, K15 KEYSW, K16 KEYSW, K17 KEYSW, K18 KEYSW, K19 KEYSW, K2 KEYSW, K20 KEYSW, K21 KEYSW, K22 KEYSW, K23 KEYSW, K24 KEYSW, K25 KEYSW, K26 KEYSW, K27 KEYSW, K28 KEYSW, K29 KEYSW, K3 KEYSW, K30 KEYSW, K31 KEYSW, K32 KEYSW, K33 KEYSW, K34 KEYSW, K35 KEYSW, K36 KEYSW, K37 KEYSW, K38 KEYSW, K39 KEYSW, K4 KEYSW, K40 KEYSW, K41 KEYSW, K42 KEYSW, K43 KEYSW, K44 KEYSW, K45 KEYSW, K5 KEYSW, K6 KEYSW, K7 KEYSW, K8 KEYSW, K9 KEYSW, SW1 SW_PUSH, U1 ATMEGA32U4, X1 XTAL_GND

Commit message: init design
Parts:
- C1, C2, C3, C4, C5, C6, C7, C8, D1, D10, D11, D12, D13, D14, D15, D16, D17, D18, D19, D2, D20, D21, D22, D23, D24, D25, D26, D27, D28, D29, D3, D30, D31, D32, D33, D34, D35, D36, D37, D38, D39, D4, D40, D41, D42, D43, D44, D45, D5, D6, D7, D8, D9, J1, R1, R2, R3, R4, SW1, U1, X1: moved to B.Cu
- moved C7 279.5 mm to (358.0, -231.0)
- moved C6 276.1 mm to (358.0, -227.8)
- moved C5 272.8 mm to (358.0, -224.6)
- moved C8 262.4 mm to (338.1, -239.7)
- moved R2 259.3 mm to (358.8, -237.3)
- moved C4 258.8 mm to (350.1, -237.3)
- moved R1 208.8 mm to (302.4, -233.4), turned to 270 degrees
- moved R3 205.2 mm to (307.2, -234.9), turned to 180 degrees
- moved X1 183.2 mm to (337.2, -228.8), turned to 45 degrees
- moved C3 158.1 mm to (345.4, -237.3)
- moved C2 146.0 mm to (337.3, -224.6), turned to 180 degrees
- moved U1 135.3 mm to (347.7, -228.6), turned to 90 degrees
- moved C1 124.3 mm to (337.2, -232.6), turned to 180 degrees
- moved R4 102.3 mm to (315.1, -228.6), turned to 270 degrees
- moved SW1 84.0 mm to (308.0, -227.8)
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